Commit message: Commenting

File: src/urdf_2dof/urdf/2dof.urdf (robot description, URDF)
Before this commit: robot urdf_2dof, 4 links, 3 joints
Links:
- link base_link: mass 0.0512057504117312 -> 0

Commit message: commentedPendulumnode+pinv->inv

File: src/urdf_2dof/urdf/2dof.urdf (robot description, URDF)
Before this commit: robot urdf_2dof, 4 links, 3 joints
Links:
- link base_link: mass 0 -> 0.0512057504117312
